File: Wearable Alert Device Schematics/Old Design/Microphone_System/Microphone_System.kicad_sch (KiCad schematic)
At the start: 15 parts

Commit message: Old Designs
Parts:
- removed Arduino_Nano_ESP1: (no value), symbol CCEW Wearable Alert:Arduino_Nano_ESP32
- removed Gravity_Reciever_Module1: (no value), symbol CCEW Wearable Alert:MIC2288
- removed LIPO_Charger1: (no value), symbol CCEW Wearable Alert Library:LIPO_Charger
- removed MEMS_Microphone_Analog1: (no value), symbol CCEW Wearable Alert Library:Fermion{colon}_MEMS_Microphone
- removed Push_Switch1: (no value), symbol CCEW Wearable Alert:320E11RED
- added Arduino_Nano_ESP: (no value), symbol CCEW Wearable Alert:Arduino_Nano_ESP32
- added I2S_MEMS_Mic: (no value), symbol CCEW Wearable Alert:I2S_MEMS_Microphone
- added Push_Switch: (no value), symbol CCEW Wearable Alert:320E11RED
- added U1: (no value), Adafruit MicroLipo Charger v2:SOT23-5, symbol Adafruit MicroLipo Charger v2-eagle-import:MCP73831/2
Connections:
- net 3.7V: now also U1.3 (VBAT)
- net GND: now also C1.1, Arduino_Nano_ESP.14 (GND), Arduino_Nano_ESP.19 (GND), I2S_MEMS_Mic. (DO), Push_Switch.3; no longer C1.2
- net Vin: now reaches 5.62k1.1, C3.1, D1.1 (K)
- net Vin: now also Arduino_Nano_ESP.15 (VIN)
- net D9: now reaches R2.2
- net D9: now also Arduino_Nano_ESP.27 (D9)
- new net 3V3: Arduino_Nano_ESP.2 (+3V3), C1.2, I2S_MEMS_Mic. (DO)
- new net D2: Arduino_Nano_ESP.20 (D2), I2S_MEMS_Mic. (DO)
- new net D3: Arduino_Nano_ESP.21 (D3), I2S_MEMS_Mic. (DO)
- new net D4: Arduino_Nano_ESP.22 (D4), I2S_MEMS_Mic. (DO)
- new net D5: Arduino_Nano_ESP.23 (D5), I2S_MEMS_Mic. (DO)
- new net D8: Arduino_Nano_ESP.26 (D8), Push_Switch.1
Other:
- note removed: "GPS Tracking"
