File: Wearable Alert Device Schematics/Old Design/Microphone_System_Wiring/Microphone_System_Wiring.kicad_sch (KiCad schematic)
At the start: 15 parts

Commit message: Old Designs
Parts:
- removed Gravity_Reciever_Module1: (no value), symbol CCEW Wearable Alert:MIC2288
- removed LIPO_Charger1: (no value), symbol CCEW Wearable Alert Library:LIPO_Charger
- removed MEMS_Microphone_Analog1: (no value), symbol CCEW Wearable Alert Library:Fermion{colon}_MEMS_Microphone
- added I2S_MEMS_Mic1: (no value), symbol CCEW Wearable Alert:I2S_MEMS_Microphone
- added U1: (no value), Adafruit MicroLipo Charger v2:SOT23-5, symbol Adafruit MicroLipo Charger v2-eagle-import:MCP73831/2
Connections:
- net 3.7V: now also U1.3 (VBAT)
- net GND: now also C1.1, I2S_MEMS_Mic1. (DO); no longer C1.2
- net at Arduino_Nano_ESP1.2 (+3V3): now also C1.2, I2S_MEMS_Mic1. (DO); no longer C1.1
- net at Arduino_Nano_ESP1.20 (D2): now also I2S_MEMS_Mic1. (DO)
- net at Arduino_Nano_ESP1.21 (D3): now also I2S_MEMS_Mic1. (DO)
- net at Arduino_Nano_ESP1.22 (D4): now also I2S_MEMS_Mic1. (DO)
- net at Arduino_Nano_ESP1.23 (D5): now also I2S_MEMS_Mic1. (DO)
Other:
- note removed: "GPS Tracking"
