File: KiCad Files/Wearable Alert Device Schematics/WearableAlertDevice_Final/WearableAlertDevice_Final.kicad_sch (KiCad schematic)
At the start: 8 parts

Commit message: Change Symbol for Lipo Charger
Parts:
- removed Adafruit_4410: (no value), symbol CCEW Wearable Alert Library:LIPO_Charger
- added LIPO_Charger: (no value), symbol CCEW Wearable Alert Library:LIPO_Charger
- renumbered MICC2288 to MIC2288
Connections:
- net 3.7V: now also LIPO_Charger.6 (JST); no longer Arduino_Nano_ESP.15 (VIN)
- net GND: now also LIPO_Charger.4 (GND)
- new net: Arduino_Nano_ESP.15 (VIN), LIPO_Charger.5 (BAT)
Changed lines of the file:
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@@
 		(color 0 0 0 0)
 	)
-	(junction
-		(at 162.56 64.77)
-		(diameter 0)
-		(color 0 0 0 0)
-	)
-	(wire
-		(pts
-			(xy 162.56 59.69) (xy 162.56 64.77)
-		)
-		(stroke
-			(width 0)
-			(type default)
-		)
-	)
-	(wire
-		(pts
-			(xy 238.76 64.77) (xy 238.76 151.13)
-		)
-		(stroke
-			(width 0)
-			(type default)
-		)
-	)
-	(wire
-		(pts
-			(xy 162.56 64.77) (xy 154.94 64.77)
+	(wire
+		(pts
+			(xy 238.76 59.69) (xy 238.76 151.13)
 		)
 		(stroke
@@
 	(wire
 		(pts
-			(xy 227.33 67.31) (xy 227.33 81.28)
-		)
-		(stroke
-			(width 0)
-			(type default)
-		)
-	)
-	(wire
-		(pts
-			(xy 154.94 67.31) (xy 227.33 67.31)
+			(xy 137.16 60.96) (xy 137.16 64.77)
 		)
 		(stroke
@@
 	(wire
 		(pts
-			(xy 162.56 64.77) (xy 238.76 64.77)
-		)
-		(stroke
-			(width 0)
-			(type default)
-		)
-	)
-	(wire
-		(pts
 			(xy 175.26 111.76) (xy 175.26 121.92)
 		)
@@
 	(wire
 		(pts
+			(xy 158.75 62.23) (xy 227.33 62.23)
+		)
+		(stroke
+			(width 0)
+			(type default)
+		)
+	)
+	(wire
+		(pts
 			(xy 87.63 123.19) (xy 101.6 123.19)
 		)
@@
 	(wire
 		(pts
+			(xy 137.16 64.77) (xy 144.78 64.77)
+		)
+		(stroke
+			(width 0)
+			(type default)
+		)
+	)
+	(wire
+		(pts
 			(xy 102.87 99.06) (xy 115.57 99.06)
 		)
@@
 	(wire
 		(pts
+			(xy 227.33 62.23) (xy 227.33 81.28)
+		)
+		(stroke
+			(width 0)
+			(type default)
+		)
+	)
+	(wire
+		(pts
 			(xy 109.22 134.62) (xy 129.54 134.62)
 		)
@@
 	(wire
 		(pts
+			(xy 158.75 59.69) (xy 238.76 59.69)
+		)
+		(stroke
+			(width 0)
+			(type default)
+		)
+	)
+	(wire
+		(pts
 			(xy 165.1 111.76) (xy 175.26 111.76)
 		)
@@
 			(width 0)
 			(type default)
-		)
-	)
-	(symbol
-		(lib_id "CCEW Wearable Alert Library:LIPO_Charger")
-		(at 152.4 76.2 90)
-		(unit 1)
-		(body_style 1)
-		(exclude_from_sim no)
-		(in_bom yes)
-		(on_board yes)
-		(in_pos_files yes)
-		(dnp no)
-		(fields_autoplaced yes)
-		(property "Reference" "Adafruit_4410"
-			(at 149.225 60.96 90)
-			(show_name no)
-			(do_not_autoplace no)
-			(effects
-				(font
-					(size 1.27 1.27)
-				)
-			)
-		)
-		(property "Value" ""
-			(at 152.4 76.2 0)
-			(show_name no)
-			(do_not_autoplace no)
-			(effects
-				(font
-					(size 1.27 1.27)
-				)
-			)
-		)
-		(property "Footprint" ""
-			(at 152.4 76.2 0)
-			(hide yes)
-			(show_name no)
-			(do_not_autoplace no)
-			(effects
-				(font
-					(size 1.27 1.27)
-				)
-			)
-		)
-		(property "Datasheet" ""
-			(at 152.4 76.2 0)
-			(hide yes)
-			(show_name no)
-			(do_not_autoplace no)
-			(effects
-				(font
-					(size 1.27 1.27)
-				)
-			)
-		)
-		(property "Description" ""
-			(at 152.4 76.2 0)
-			(hide yes)
-			(show_name no)
-			(do_not_autoplace no)
-			(effects
-				(font
-					(size 1.27 1.27)
-				)
-			)
-		)
-		(pin "4"
-		)
-		(pin "5"
-		)
-		(pin "3"
-		)
-		(pin "1"
-		)
-		(pin "2"
-		)
-		(instances
-			(project "WearableAlertDevice_Final"
-				(path "/b3918005-f5d6-4a88-9e4d-fb74a34c57a0"
-					(reference "Adafruit_4410")
-					(unit 1)
-				)
-			)
 		)
 	)
@@
 		(in_pos_files yes)
 		(dnp no)
-		(property "Reference" "MICC2288"
+		(property "Reference" "MIC2288"
 			(at 101.346 90.424 90)
 			(show_name no)
@@
 			(project "WearableAlertDevice_Final"
 				(path "/b3918005-f5d6-4a88-9e4d-fb74a34c57a0"
-					(reference "MICC2288")
+					(reference "MIC2288")
+					(unit 1)
+				)
+			)
+		)
+	)
+	(symbol
+		(lib_name "LIPO_Charger_1")
+		(lib_id "CCEW Wearable Alert Library:LIPO_Charger")
+		(at 156.21 71.12 90)
+		(unit 1)
+		(body_style 1)
+		(exclude_from_sim no)
+		(in_bom yes)
+		(on_board yes)
+		(in_pos_files yes)
+		(dnp no)
+		(fields_autoplaced yes)
+		(property "Reference" "LIPO_Charger"
+			(at 151.765 55.88 90)
+			(show_name no)
+			(do_not_autoplace no)
+			(effects
+				(font
+					(size 1.27 1.27)
+				)
+			)
+		)
+		(property "Value" ""
+			(at 156.21 71.12 0)
+			(show_name no)
+			(do_not_autoplace no)
+			(effects
+				(font
+					(size 1.27 1.27)
+				)
+			)
+		)
+		(property "Footprint" ""
+			(at 156.21 71.12 0)
+			(hide yes)
+			(show_name no)
+			(do_not_autoplace no)
+			(effects
+				(font
+					(size 1.27 1.27)
+				)
+			)
+		)
+		(property "Datasheet" ""
+			(at 156.21 71.12 0)
+			(hide yes)
+			(show_name no)
+			(do_not_autoplace no)
+			(effects
+				(font
+					(size 1.27 1.27)
+				)
+			)
+		)
+		(property "Description" "LIPOLY BATTERY CHARGER W/USB C"
+			(at 156.21 71.12 0)
+			(hide yes)
+			(show_name no)
+			(do_not_autoplace no)
+			(effects
+				(font
+					(size 1.27 1.27)
+				)
+			)
+		)
+		(pin "5"
+		)
+		(pin "6"
+		)
+		(pin "4"
+		)
+		(pin "1"
+		)
+		(pin "2"
+		)
+		(pin "3"
+		)
+		(instances
+			(project "WearableAlertDevice_Final"
+				(path "/b3918005-f5d6-4a88-9e4d-fb74a34c57a0"
+					(reference "LIPO_Charger")
 					(unit 1)
 				)
@@
 	(symbol
 		(lib_id "power:VCC")
-		(at 162.56 59.69 0)
+		(at 137.16 60.96 0)
 		(unit 1)
 		(body_style 1)
@@
 		(dnp no)
 		(property "Reference" "#PWR01"
-			(at 162.56 63.5 0)
+			(at 137.16 64.77 0)
 			(hide yes)
 			(show_name no)
@@
 		)
 		(property "Value" "3.7V"
-			(at 160.528 55.372 0)
+			(at 135.128 56.642 0)
 			(show_name no)
 			(do_not_autoplace no)
@@
 		)
 		(property "Footprint" ""
-			(at 162.56 59.69 0)
+			(at 137.16 60.96 0)
 			(hide yes)
 			(show_name no)
@@
 		)
 		(property "Datasheet" ""
-			(at 162.56 59.69 0)
+			(at 137.16 60.96 0)
 			(hide yes)
 			(show_name no)
@@
 		)
 		(property "Description" "Power symbol creates a global label with name \"VCC\""
-			(at 162.56 59.69 0)
-			(hide yes)
-			(show_name no)
+			(at 137.16 60.96 0)
+			(hide yes)
+			(show_name no)

Commit message: Updated GPS Name
Parts:
- renumbered MIC2288 to Gravity_GNSS_Receiver_Module
Changed lines of the file:
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@@
 	(paper "A4")
+	(junction
+		(at 123.19 104.14)
+		(diameter 0)
+		(color 0 0 0 0)
+	)
+	(junction
+		(at 227.33 135.89)
+		(diameter 0)
+		(color 0 0 0 0)
+	)
+	(junction
+		(at 227.33 97.79)
+		(diameter 0)
+		(color 0 0 0 0)
+	)
+	(junction
+		(at 109.22 134.62)
+		(diameter 0)
+		(color 0 0 0 0)
+	)
+	(junction
+		(at 186.69 135.89)
+		(diameter 0)
+		(color 0 0 0 0)
+	)
 	(junction
 		(at 227.33 81.28)
@@
 	)
 	(junction
-		(at 123.19 104.14)
-		(diameter 0)
-		(color 0 0 0 0)
-	)
-	(junction
-		(at 227.33 135.89)
-		(diameter 0)
-		(color 0 0 0 0)
-	)
-	(junction
-		(at 227.33 97.79)
-		(diameter 0)
-		(color 0 0 0 0)
-	)
-	(junction
-		(at 109.22 134.62)
-		(diameter 0)
-		(color 0 0 0 0)
-	)
-	(junction
-		(at 186.69 135.89)
-		(diameter 0)
-		(color 0 0 0 0)
-	)
-	(junction
 		(at 227.33 121.92)
 		(diameter 0)
@@
 	(wire
 		(pts
-			(xy 109.22 81.28) (xy 227.33 81.28)
+			(xy 114.3 81.28) (xy 227.33 81.28)
 		)
 		(stroke
@@
 	(wire
 		(pts
-			(xy 102.87 96.52) (xy 109.22 96.52)
+			(xy 102.87 96.52) (xy 114.3 96.52)
 		)
 		(stroke
@@
 	(wire
 		(pts
-			(xy 109.22 96.52) (xy 109.22 81.28)
+			(xy 114.3 96.52) (xy 114.3 81.28)
 		)
 		(stroke
@@
 		(in_pos_files yes)
 		(dnp no)
-		(property "Reference" "MIC2288"
-			(at 101.346 90.424 90)
+		(property "Reference" "Gravity_GNSS_Receiver_Module"
+			(at 109.982 89.662 90)
 			(show_name no)
 			(do_not_autoplace no)
@@
 			(project "WearableAlertDevice_Final"
 				(path "/b3918005-f5d6-4a88-9e4d-fb74a34c57a0"
-					(reference "MIC2288")
+					(reference "Gravity_GNSS_Receiver_Module")
 					(unit 1)
 				)

Commit message: Add Team Names, Date, and Project name
Other:
- company: (none) -> CCEW
- title: (none) -> Wearable Alert Device Schematics
Changed lines of the file:
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@@
 	(generator_version "10.0")
 	(paper "A4")
+	(title_block
+		(title "Wearable Alert Device Schematics")
+		(date "2026-05-04")
+		(company "CCEW")
+		(comment 1 "Team Members: Jonas Wallman, Ryan Kiesau, Cody Chan, Alex Ho")
+	)
 	(junction
 		(at 123.19 104.14)
